Commit message: weaken op3 max effort

File: gym_op3/urdf/robotis_op3.structure.head.xacro (robot description, xacro)
@@ -12,5 +12,5 @@
     <origin xyz="-0.001 0.0 0.1365" rpy="0 0 0" />
     <axis xyz="0 0 1" />
-    <limit effort="1000" velocity="100" lower="${-pi*0.9}" upper="${pi*0.9}" />
+    <limit effort="10" velocity="100" lower="${-pi*0.9}" upper="${pi*0.9}" />
     <dynamics damping="0.1" friction="0.0" />
   </joint>
@@ -34,5 +34,5 @@
     <origin xyz="0.010 0.019 0.0285" rpy="0 0 0" />
     <axis xyz="0 -1 0" />
-    <limit effort="1000" velocity="100" lower="${-pi*0.9}" upper="${pi*0.9}" />
+    <limit effort="10" velocity="100" lower="${-pi*0.9}" upper="${pi*0.9}" />
     <dynamics damping="0.1" friction="0.0" />
   </joint>

File: gym_op3/urdf/robotis_op3.structure.larm.xacro (robot description, xacro)
@@ -12,5 +12,5 @@
     <origin xyz="-0.001 0.06 0.111" rpy="0 0 0" />
     <axis xyz="0 1 0" />
-    <limit effort="1000" velocity="100" lower="${-pi*0.9}" upper="${pi*0.9}" />
+    <limit effort="10" velocity="100" lower="${-pi*0.9}" upper="${pi*0.9}" />
     <dynamics damping="0.1" friction="0.0" />
   </joint>
@@ -34,5 +34,5 @@
     <origin xyz="0.019 0.0285 -0.010" rpy="0 0 0" />
     <axis xyz="-1 0 0" />
-    <limit effort="1000" velocity="100" lower="${-pi*0.9}" upper="${pi*0.9}" />
+    <limit effort="10" velocity="100" lower="${-pi*0.9}" upper="${pi*0.9}" />
     <dynamics damping="0.1" friction="0.0" />
   </joint>
@@ -56,5 +56,5 @@
     <origin xyz="0.0 0.0904 -0.0001" rpy="0 0 0" />
     <axis xyz="1 0 0" />
-    <limit effort="1000" velocity="100" lower="${-pi*0.9}" upper="${pi*0.9}" />
+    <limit effort="10" velocity="100" lower="${-pi*0.9}" upper="${pi*0.9}" />
     <dynamics damping="0.1" friction="0.0" />
   </joint>

File: gym_op3/urdf/robotis_op3.structure.lleg.xacro (robot description, xacro)
@@ -12,5 +12,5 @@
     <origin xyz="0.0 0.035 0.0" rpy="0 0 0" />
     <axis xyz="0 0 -1" />
-    <limit effort="1000" velocity="100" lower="${-pi*0.9}" upper="${pi*0.9}" />
+    <limit effort="10" velocity="100" lower="${-pi*0.9}" upper="${pi*0.9}" />
     <dynamics damping="0.1" friction="0.0" />
   </joint>
@@ -34,5 +34,5 @@
     <origin xyz="-0.024 0.0 -0.0285" rpy="0 0 0" />
     <axis xyz="-1 0 0" />
-    <limit effort="1000" velocity="100" lower="${-pi*0.9}" upper="${pi*0.9}" />
+    <limit effort="10" velocity="100" lower="${-pi*0.9}" upper="${pi*0.9}" />
     <dynamics damping="0.1" friction="0.0" />
   </joint>
@@ -56,5 +56,5 @@
     <origin xyz="0.0241 0.019 0.0" rpy="0 0 0" />
     <axis xyz="0 1 0" />
-    <limit effort="1000" velocity="100" lower="${-pi*0.9}" upper="${pi*0.9}" />
+    <limit effort="10" velocity="100" lower="${-pi*0.9}" upper="${pi*0.9}" />
     <dynamics damping="0.1" friction="0.0" />
   </joint>
@@ -78,5 +78,5 @@
     <origin xyz="0.0 0.0 -0.11015" rpy="0 0 0" />
     <axis xyz="0 1 0" />
-    <limit effort="1000" velocity="100" lower="${-pi*0.9}" upper="${pi*0.9}" />
+    <limit effort="10" velocity="100" lower="${-pi*0.9}" upper="${pi*0.9}" />
     <dynamics damping="0.1" friction="0.0" />
   </joint>
@@ -100,5 +100,5 @@
     <origin xyz="0 0 -0.110" rpy="0 0 0" />
     <axis xyz="0 -1 0" />
-    <limit effort="1000" velocity="100" lower="${-pi*0.9}" upper="${pi*0.9}" />
+    <limit effort="10" velocity="100" lower="${-pi*0.9}" upper="${pi*0.9}" />
     <dynamics damping="0.1" friction="0.0" />
   </joint>
@@ -122,5 +122,5 @@
     <origin xyz="-0.0241 -0.019 0" rpy="0 0 0" />
     <axis xyz="1 0 0" />
-    <limit effort="1000" velocity="100" lower="${-pi*0.9}" upper="${pi*0.9}" />
+    <limit effort="10" velocity="100" lower="${-pi*0.9}" upper="${pi*0.9}" />
     <dynamics damping="0.1" friction="0.0" />
   </joint>

File: gym_op3/urdf/robotis_op3.structure.rarm.xacro (robot description, xacro)
@@ -12,5 +12,5 @@
     <origin xyz="-0.001 -0.06 0.111" rpy="0 0 0" />
     <axis xyz="0 -1 0" />
-    <limit effort="1000" velocity="100" lower="${-pi*0.9}" upper="${pi*0.9}" />
+    <limit effort="10" velocity="100" lower="${-pi*0.9}" upper="${pi*0.9}" />
     <dynamics damping="0.1" friction="0.0" />
   </joint>
@@ -34,5 +34,5 @@
     <origin xyz="0.019 -0.0285 -0.010" rpy="0 0 0" />
     <axis xyz="-1 0 0" />
-    <limit effort="1000" velocity="100" lower="${-pi*0.9}" upper="${pi*0.9}" />
+    <limit effort="10" velocity="100" lower="${-pi*0.9}" upper="${pi*0.9}" />
     <dynamics damping="0.1" friction="0.0" />
   </joint>
@@ -56,5 +56,5 @@
     <origin xyz="0.0 -0.0904 -0.0001" rpy="0 0 0" />
     <axis xyz="1 0 0" />
-    <limit effort="1000" velocity="100" lower="${-pi*0.9}" upper="${pi*0.9}" />
+    <limit effort="10" velocity="100" lower="${-pi*0.9}" upper="${pi*0.9}" />
     <dynamics damping="0.1" friction="0.0" />
   </joint>

File: gym_op3/urdf/robotis_op3.structure.rleg.xacro (robot description, xacro)
@@ -12,5 +12,5 @@
     <origin xyz="0.0 -0.035 0.0" rpy="0 0 0" />
     <axis xyz="0 0 -1" />
-    <limit effort="1000" velocity="100" lower="${-pi*0.9}" upper="${pi*0.9}" />
+    <limit effort="10" velocity="100" lower="${-pi*0.9}" upper="${pi*0.9}" />
     <dynamics damping="0.1" friction="0.0" />
   </joint>
@@ -34,5 +34,5 @@
     <origin xyz="-0.024 0.0 -0.0285" rpy="0 0 0" />
     <axis xyz="-1 0 0" />
-    <limit effort="1000" velocity="100" lower="${-pi*0.9}" upper="${pi*0.9}" />
+    <limit effort="10" velocity="100" lower="${-pi*0.9}" upper="${pi*0.9}" />
     <dynamics damping="0.1" friction="0.0" />
   </joint>
@@ -56,5 +56,5 @@
     <origin xyz="0.0241 -0.019 0.0" rpy="0 0 0" />
     <axis xyz="0 -1 0" />
-    <limit effort="1000" velocity="100" lower="${-pi*0.9}" upper="${pi*0.9}" />
+    <limit effort="10" velocity="100" lower="${-pi*0.9}" upper="${pi*0.9}" />
     <dynamics damping="0.1" friction="0.0" />
   </joint>
@@ -78,5 +78,5 @@
     <origin xyz="0.0 0.0 -0.11015" rpy="0 0 0" />
     <axis xyz="0 -1 0" />
-    <limit effort="1000" velocity="100" lower="${-pi*0.9}" upper="${pi*0.9}" />
+    <limit effort="10" velocity="100" lower="${-pi*0.9}" upper="${pi*0.9}" />
     <dynamics damping="0.1" friction="0.0" />
   </joint>
@@ -100,5 +100,5 @@
     <origin xyz="0 0 -0.110" rpy="0 0 0" />
     <axis xyz="0 1 0" />
-    <limit effort="1000" velocity="100" lower="${-pi*0.9}" upper="${pi*0.9}" />
+    <limit effort="10" velocity="100" lower="${-pi*0.9}" upper="${pi*0.9}" />
     <dynamics damping="0.1" friction="0.0" />
   </joint>
@@ -122,5 +122,5 @@
     <origin xyz="-0.0241 0.019 0" rpy="0 0 0" />
     <axis xyz="1 0 0" />
-    <limit effort="1000" velocity="100" lower="${-pi*0.9}" upper="${pi*0.9}" />
+    <limit effort="10" velocity="100" lower="${-pi*0.9}" upper="${pi*0.9}" />
     <dynamics damping="0.1" friction="0.0" />
   </joint>

Commit message: weaken damping

File: gym_op3/urdf/robotis_op3.structure.head.xacro (robot description, xacro)
@@ -13,5 +13,5 @@
     <axis xyz="0 0 1" />
     <limit effort="10" velocity="100" lower="${-pi*0.9}" upper="${pi*0.9}" />
-    <dynamics damping="0.1" friction="0.0" />
+    <dynamics damping="0.01" friction="0.0" />
   </joint>
   <xacro:insert_transmission name="head_pan" />
@@ -35,5 +35,5 @@
     <axis xyz="0 -1 0" />
     <limit effort="10" velocity="100" lower="${-pi*0.9}" upper="${pi*0.9}" />
-    <dynamics damping="0.1" friction="0.0" />
+    <dynamics damping="0.01" friction="0.0" />
   </joint>
   <xacro:insert_transmission name="head_tilt" />

File: gym_op3/urdf/robotis_op3.structure.larm.xacro (robot description, xacro)
@@ -13,5 +13,5 @@
     <axis xyz="0 1 0" />
     <limit effort="10" velocity="100" lower="${-pi*0.9}" upper="${pi*0.9}" />
-    <dynamics damping="0.1" friction="0.0" />
+    <dynamics damping="0.01" friction="0.0" />
   </joint>
   <xacro:insert_transmission name="l_sho_pitch" />
@@ -35,5 +35,5 @@
     <axis xyz="-1 0 0" />
     <limit effort="10" velocity="100" lower="${-pi*0.9}" upper="${pi*0.9}" />
-    <dynamics damping="0.1" friction="0.0" />
+    <dynamics damping="0.01" friction="0.0" />
   </joint>
   <xacro:insert_transmission name="l_sho_roll" />
@@ -57,5 +57,5 @@
     <axis xyz="1 0 0" />
     <limit effort="10" velocity="100" lower="${-pi*0.9}" upper="${pi*0.9}" />
-    <dynamics damping="0.1" friction="0.0" />
+    <dynamics damping="0.01" friction="0.0" />
   </joint>
   <xacro:insert_transmission name="l_el" />

File: gym_op3/urdf/robotis_op3.structure.lleg.xacro (robot description, xacro)
@@ -13,5 +13,5 @@
     <axis xyz="0 0 -1" />
     <limit effort="10" velocity="100" lower="${-pi*0.9}" upper="${pi*0.9}" />
-    <dynamics damping="0.1" friction="0.0" />
+    <dynamics damping="0.01" friction="0.0" />
   </joint>
   <xacro:insert_transmission name="l_hip_yaw" />
@@ -35,5 +35,5 @@
     <axis xyz="-1 0 0" />
     <limit effort="10" velocity="100" lower="${-pi*0.9}" upper="${pi*0.9}" />
-    <dynamics damping="0.1" friction="0.0" />
+    <dynamics damping="0.01" friction="0.0" />
   </joint>
   <xacro:insert_transmission name="l_hip_roll" />
@@ -57,5 +57,5 @@
     <axis xyz="0 1 0" />
     <limit effort="10" velocity="100" lower="${-pi*0.9}" upper="${pi*0.9}" />
-    <dynamics damping="0.1" friction="0.0" />
+    <dynamics damping="0.01" friction="0.0" />
   </joint>
   <xacro:insert_transmission name="l_hip_pitch" />
@@ -79,5 +79,5 @@
     <axis xyz="0 1 0" />
     <limit effort="10" velocity="100" lower="${-pi*0.9}" upper="${pi*0.9}" />
-    <dynamics damping="0.1" friction="0.0" />
+    <dynamics damping="0.01" friction="0.0" />
   </joint>
   <xacro:insert_transmission name="l_knee" />
@@ -101,5 +101,5 @@
     <axis xyz="0 -1 0" />
     <limit effort="10" velocity="100" lower="${-pi*0.9}" upper="${pi*0.9}" />
-    <dynamics damping="0.1" friction="0.0" />
+    <dynamics damping="0.01" friction="0.0" />
   </joint>
   <xacro:insert_transmission name="l_ank_pitch" />
@@ -123,5 +123,5 @@
     <axis xyz="1 0 0" />
     <limit effort="10" velocity="100" lower="${-pi*0.9}" upper="${pi*0.9}" />
-    <dynamics damping="0.1" friction="0.0" />
+    <dynamics damping="0.01" friction="0.0" />
   </joint>
   <xacro:insert_transmission name="l_ank_roll" />

File: gym_op3/urdf/robotis_op3.structure.rarm.xacro (robot description, xacro)
@@ -13,5 +13,5 @@
     <axis xyz="0 -1 0" />
     <limit effort="10" velocity="100" lower="${-pi*0.9}" upper="${pi*0.9}" />
-    <dynamics damping="0.1" friction="0.0" />
+    <dynamics damping="0.01" friction="0.0" />
   </joint>
   <xacro:insert_transmission name="r_sho_pitch" />
@@ -35,5 +35,5 @@
     <axis xyz="-1 0 0" />
     <limit effort="10" velocity="100" lower="${-pi*0.9}" upper="${pi*0.9}" />
-    <dynamics damping="0.1" friction="0.0" />
+    <dynamics damping="0.01" friction="0.0" />
   </joint>
   <xacro:insert_transmission name="r_sho_roll" />
@@ -57,5 +57,5 @@
     <axis xyz="1 0 0" />
     <limit effort="10" velocity="100" lower="${-pi*0.9}" upper="${pi*0.9}" />
-    <dynamics damping="0.1" friction="0.0" />
+    <dynamics damping="0.01" friction="0.0" />
   </joint>
   <xacro:insert_transmission name="r_el" />

File: gym_op3/urdf/robotis_op3.structure.rleg.xacro (robot description, xacro)
@@ -13,5 +13,5 @@
     <axis xyz="0 0 -1" />
     <limit effort="10" velocity="100" lower="${-pi*0.9}" upper="${pi*0.9}" />
-    <dynamics damping="0.1" friction="0.0" />
+    <dynamics damping="0.01" friction="0.0" />
   </joint>
   <xacro:insert_transmission name="r_hip_yaw" />
@@ -35,5 +35,5 @@
     <axis xyz="-1 0 0" />
     <limit effort="10" velocity="100" lower="${-pi*0.9}" upper="${pi*0.9}" />
-    <dynamics damping="0.1" friction="0.0" />
+    <dynamics damping="0.01" friction="0.0" />
   </joint>
   <xacro:insert_transmission name="r_hip_roll" />
@@ -57,5 +57,5 @@
     <axis xyz="0 -1 0" />
     <limit effort="10" velocity="100" lower="${-pi*0.9}" upper="${pi*0.9}" />
-    <dynamics damping="0.1" friction="0.0" />
+    <dynamics damping="0.01" friction="0.0" />
   </joint>
   <xacro:insert_transmission name="r_hip_pitch" />
@@ -79,5 +79,5 @@
     <axis xyz="0 -1 0" />
     <limit effort="10" velocity="100" lower="${-pi*0.9}" upper="${pi*0.9}" />
-    <dynamics damping="0.1" friction="0.0" />
+    <dynamics damping="0.01" friction="0.0" />
   </joint>
   <xacro:insert_transmission name="r_knee" />
@@ -101,5 +101,5 @@
     <axis xyz="0 1 0" />
     <limit effort="10" velocity="100" lower="${-pi*0.9}" upper="${pi*0.9}" />
-    <dynamics damping="0.1" friction="0.0" />
+    <dynamics damping="0.01" friction="0.0" />
   </joint>
   <xacro:insert_transmission name="r_ank_pitch" />
@@ -123,5 +123,5 @@
     <axis xyz="1 0 0" />
     <limit effort="10" velocity="100" lower="${-pi*0.9}" upper="${pi*0.9}" />
-    <dynamics damping="0.1" friction="0.0" />
+    <dynamics damping="0.01" friction="0.0" />
   </joint>
   <xacro:insert_transmission name="r_ank_roll" />
