Commit message: Remove unused link, joint of camera in URDF

File: gym_op3/urdf/robotis_op3.gazebo.xacro (robot description, xacro)
@@ -227,5 +227,5 @@
 -->
   <!-- head camera -->
-  <gazebo reference="cam_gazebo_link">
+  <!-- <gazebo reference="cam_gazebo_link">
     <sensor name='camera' type='camera'>
       <pose>-0.050000 -0.010000 0.000000 -1.5708 0.000000 -3.141592</pose>
@@ -259,5 +259,5 @@
       </plugin>
     </sensor>
-  </gazebo>
+  </gazebo> -->
   <!-- imu sensor -->
   <gazebo reference="body_link">

File: gym_op3/urdf/robotis_op3.structure.head.xacro (robot description, xacro)
@@ -51,20 +51,20 @@
   </link>
   <!-- camera joint -->
-  <joint name="cam" type="fixed">
+  <!-- <joint name="cam" type="fixed">
     <origin xyz="0.01425 -0.019 0.04975" rpy="${-pi*0.5} 0 ${-pi*0.5}"/>
     <parent link="head_tilt_link"/>
     <child link="cam_link"/>
-  </joint>
-  <joint name="cam_gazebo" type="fixed">
+  </joint> -->
+  <!-- <joint name="cam_gazebo" type="fixed">
     <origin xyz="0.01425 -0.019 0.04975" rpy="0 0 0"/>
     <parent link="head_tilt_link"/>
     <child link="cam_gazebo_link"/>
-  </joint>
+  </joint> -->
   <!-- camera link -->
-  <link name="cam_link">
-  </link>
+  <!-- <link name="cam_link">
+  </link> -->
   <!-- camera link -->
-  <link name="cam_gazebo_link">
-  </link>
+  <!-- <link name="cam_gazebo_link">
+  </link> -->
   </xacro:macro>
 </robot>
